File: BMS_Temp_Board/BMS_Temp_Board/BMS_Temp_Board.kicad_sch (KiCad schematic)
At the start: 0 parts

Commit message: BMS_Temp
added mux
Parts:
- added IC1, IC2, IC3: LTC1380IGN#PBF, SOP64P601X173-16N, symbol BMS_Temp_Library:LTC1380IGN#PBF
- added R1: 100k, Resistor_SMD:R_0603_1608Metric, symbol Device:R
Connections:
- new net: IC3.6 (S5), IC3.8 (S7)
- new net: IC1.1 (S0), IC2.1 (S0)
- new net: IC1.10 (VEE), IC2.10 (VEE)
- new net: IC1.11 (GND), IC2.11 (GND)
- new net: IC1.12 (A1), IC2.12 (A1)
- new net: IC1.13 (A0), IC2.13 (A0)
- new net: IC1.14 (SDA), IC2.14 (SDA)
- new net: IC1.15 (SCL), IC2.15 (SCL)
- new net: IC1.16 (VCC), IC2.16 (VCC)
- new net: IC1.2 (S1), IC2.2 (S1)
- new net: IC1.3 (S2), IC2.3 (S2)
- new net: IC1.4 (S3), IC2.4 (S3)
- new net: IC1.5 (S4), IC2.5 (S4)
- new net: IC1.6 (S5), IC2.6 (S5)
- new net: IC1.7 (S6), IC2.7 (S6)
- new net: IC1.8 (S7), IC2.8 (S7)
- new net: IC1.9 (D0), IC2.9 (D0)
