File: BMS_Temp_Board/BMS_Temp_Board.kicad_pcb (KiCad board)
At the start: 2 copper layers, 82 parts, among them IC1 ESP32-S3-WROOM-1-N8R8, IC10 CD74HC4067PWR, IC11 CD74HC4067PWR, IC12 CD74HC4067PWR, IC13 CD74HC4067PWR, IC14 CD74HC4067PWR, IC15 CD74HC4067PWR, IC16 CD74HC4067PWR, IC17 CD74HC4067PWR, IC18 CD74HC4067PWR, IC19 CD74HC4067PWR, IC2 CP2102N-A02-GQFN28, IC20 CD74HC4067PWR, IC21 CD74HC4067PWR, IC22 CD74HC4067PWR, IC23 CD74HC4067PWR, IC3 CD74HC4067PWR, IC3 TLP175A_TPL,E, IC4 TPS2116DRLR, IC5 MIC37100-3.3WS, IC6 CD74HC4067PWR, IC7 CD74HC4067PWR, IC8 CD74HC4067PWR, IC9 CD74HC4067PWR, J1 ESP_USB, J10 B32B-PUDSS-1_LF__SN_, J11 B32B-PUDSS-1_LF__SN_, J12 B32B-PUDSS-1_LF__SN_, J13 B32B-PUDSS-1_LF__SN_, J14 B32B-PUDSS-1_LF__SN_, J15 B32B-PUDSS-1_LF__SN_, J16 B32B-PUDSS-1_LF__SN_, J17 B32B-PUDSS-1_LF__SN_, J18 B32B-PUDSS-1_LF__SN_, J19 B32B-PUDSS-1_LF__SN_, J2 B32B-PUDSS-1_LF__SN_, J20 B32B-PUDSS-1_LF__SN_, J21 B2B-PH-K-S_LF__SN_, J3 B32B-PUDSS-1_LF__SN_, J4 B32B-PUDSS-1_LF__SN_, J5 B32B-PUDSS-1_LF__SN_, J6 B32B-PUDSS-1_LF__SN_, J7 B32B-PUDSS-1_LF__SN_, J8 B32B-PUDSS-1_LF__SN_, J9 B32B-PUDSS-1_LF__SN_, Q1 MMBT2222LT1G, Q2 MMBT2222LT1G, U1 USBLC6-2SC6, U2 SN65HVD230

Commit message: started pcb design
Parts:
- removed C11, C13: 100nF, Capacitor_SMD:C_0603_1608Metric
- removed D1: ESDCAN03-2BWY, SDM_MiscFootprint:SOT65P210X110-3N
- removed the IC3 at (44.8, 47.6)
- removed R12: 120, Resistor_SMD:R_0603_1608Metric
- removed R15: 10k, Resistor_SMD:R_0603_1608Metric
- removed U2: SN65HVD230, Package_SO:SOIC-8_3.9x4.9mm_P1.27mm
- moved J20 196.7 mm to (111.9, 37.3), turned to 90 degrees
- moved J19 182.1 mm to (134.9, 37.0), turned to 90 degrees
- moved J18 169.7 mm to (156.6, 37.1), turned to 90 degrees
- moved J17 160.6 mm to (180.2, 37.1), turned to 90 degrees
- moved J16 155.0 mm to (202.4, 37.0), turned to 90 degrees
- moved J15 153.7 mm to (225.4, 37.0), turned to 90 degrees
- moved IC6 130.1 mm to (100.0, 131.1), turned to -90 degrees
- moved IC3 116.4 mm to (122.9, 131.1), turned to -90 degrees
- moved IC7 115.0 mm to (145.5, 131.1), turned to -90 degrees
- moved IC10 114.4 mm to (213.0, 131.7), turned to -90 degrees
- moved C1 112.2 mm to (75.8, 125.4), turned to -90 degrees
- moved IC8 111.9 mm to (168.3, 131.2), turned to -90 degrees
- moved IC9 110.7 mm to (191.0, 131.4), turned to -90 degrees
- moved C2 107.9 mm to (69.2, 125.4), turned to 90 degrees
- moved C3 106.1 mm to (71.2, 125.4), turned to 90 degrees
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Connections:
- IC1 pad 31: unconnected-(IC1-IO38-Pad31) -> /USER_LED
Routing:
- net /MUX E7: track 0.00 -> 164.4 mm
- net /MUX E14: track 0.00 -> 164.2 mm
- net /MUX E6: track 0.00 -> 147.3 mm
- net /MUX E15: track 0.00 -> 140.5 mm
- net /MUX E8: track 0.00 -> 139.5 mm
- net /MUX E5: track 0.00 -> 126.1 mm
- net /MUX E16: track 0.00 -> 117.3 mm
- net /MUX E9: track 0.00 -> 116.7 mm
- net /MUX E4: track 0.00 -> 104.2 mm
- net /MUX E10: track 0.00 -> 92.7 mm
- net /MUX E17: track 0.00 -> 89.5 mm
- net /MUX E3: track 0.00 -> 82.0 mm
- net /MUX E11: track 0.00 -> 70.7 mm
- net /MUX E18: track 0.00 -> 68.1 mm
- net /MUX E2: track 0.00 -> 60.8 mm
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