File: BMS_Temp_Board/BMS_Temp_Board.kicad_sch (KiCad schematic)
At the start: 75 parts, among them IC1 ESP32-S3-WROOM-1-N8R8, IC10 CD74HC4067PWR, IC11 CD74HC4067PWR, IC12 CD74HC4067PWR, IC13 CD74HC4067PWR, IC14 CD74HC4067PWR, IC15 CD74HC4067PWR, IC16 CD74HC4067PWR, IC17 CD74HC4067PWR, IC18 CD74HC4067PWR, IC19 CD74HC4067PWR, IC2 CP2102N-A02-GQFN28, IC20 CD74HC4067PWR, IC21 CD74HC4067PWR, IC22 CD74HC4067PWR, IC23 CD74HC4067PWR, IC3 CD74HC4067PWR, IC4 TPS2116DRLR, IC5 MIC37100-3.3WS, IC6 CD74HC4067PWR, IC7 CD74HC4067PWR, IC8 CD74HC4067PWR, IC9 CD74HC4067PWR, J1 ESP_USB, J10 B32B-PUDSS-1_LF__SN_, J11 B32B-PUDSS-1_LF__SN_, J12 B32B-PUDSS-1_LF__SN_, J13 B32B-PUDSS-1_LF__SN_, J14 B32B-PUDSS-1_LF__SN_, J15 B32B-PUDSS-1_LF__SN_, J16 B32B-PUDSS-1_LF__SN_, J17 B32B-PUDSS-1_LF__SN_, J18 B32B-PUDSS-1_LF__SN_, J19 B32B-PUDSS-1_LF__SN_, J2 B32B-PUDSS-1_LF__SN_, J20 B32B-PUDSS-1_LF__SN_, J21 B2B-PH-K-S_LF__SN_, J3 B32B-PUDSS-1_LF__SN_, J4 B32B-PUDSS-1_LF__SN_, J5 B32B-PUDSS-1_LF__SN_, J6 B32B-PUDSS-1_LF__SN_, J7 B32B-PUDSS-1_LF__SN_, J8 B32B-PUDSS-1_LF__SN_, J9 B32B-PUDSS-1_LF__SN_, Q1 MMBT2222LT1G, Q2 MMBT2222LT1G, U1 USBLC6-2SC6

Commit message: started pcb design
Connections:
- net USER_LED: now also IC1.31 (IO38)
- no-connect marks 26 -> 25
Changed lines of the file:
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@@
 	)
 	(no_connect
-		(at 82.55 40.64)
-	)
-	(no_connect
 		(at 220.98 69.85)
 	)
@@
 	(wire
 		(pts
+			(xy 82.55 40.64) (xy 92.71 40.64)
+		)
+		(stroke
+			(width 0)
+			(type default)
+		)
+	)
+	(wire
+		(pts
 			(xy 257.81 265.43) (xy 279.4 265.43)
 		)
@@
 		(effects
 			(font
+				(size 1.27 1.27)
+			)
+			(justify right bottom)
+		)
+	)
+	(label "USER_LED"
+		(at 92.71 40.64 180)
+		(effects
+			(font
