File: BMS_Temp_Board/BMS_Temp_Board_V1.kicad_sch (KiCad schematic)
At the start: 77 parts, among them IC1 ESP32-S3-WROOM-1-N8R8, IC10 CD74HC4067PWR, IC11 CD74HC4067PWR, IC12 CD74HC4067PWR, IC13 CD74HC4067PWR, IC14 CD74HC4067PWR, IC15 CD74HC4067PWR, IC2 CP2102N-A02-GQFN28, IC3 TLP175A_TPL,E, IC4 TPS2116DRLR, IC5 MIC37100-3.3WS, IC6 CD74HC4067PWR, IC7 CD74HC4067PWR, IC8 CD74HC4067PWR, IC9 CD74HC4067PWR, J1 ESP_USB, J10 B32B-PUDSS-1_LF__SN_, J11 B32B-PUDSS-1_LF__SN_, J12 B2B-PH-K-S, J13 SM04B-ULHK-1TA1-ETB_HF_, J14 B2B-PH-K-S, J2 B32B-PUDSS-1_LF__SN_, J3 B32B-PUDSS-1_LF__SN_, J4 B32B-PUDSS-1_LF__SN_, J5 B32B-PUDSS-1_LF__SN_, J6 B32B-PUDSS-1_LF__SN_, J7 B32B-PUDSS-1_LF__SN_, J8 B32B-PUDSS-1_LF__SN_, J9 B32B-PUDSS-1_LF__SN_, Q1 MMBT2222LT1G, Q2 MMBT2222LT1G, U1 USBLC6-2SC6, U2 SN65HVD230, U3 LM2575HVS-5.0_NOPB

Commit message: changed C17 and some layout on bms temp
Parts:
- C17: footprint Capacitor_SMD:C_0603_1608Metric -> Capacitor_SMD:CP_Elec_10x10

Commit message: made changes from design review
Parts:
- removed J13: SM04B-ULHK-1TA1-ETB_HF_, SM04B-ULH:SM04BULHK1TA1ETBHF, symbol SM04B-ULHK-1TA1-ETB_HF_:SM04B-ULHK-1TA1-ETB_HF_
- added J15: B2B-PH-K-S, B2B_PH_K_S:JST_B2B-PH-K-S, symbol B2B-PH-K-S:B2B-PH-K-S
- added R17, R18, R19, R20, R21, R22, R23, R24, R25, R26: 10k, Resistor_SMD:R_0603_1608Metric, symbol Device:R
- C15: footprint Capacitor_SMD:C_0603_1608Metric -> 865080545012:WCAP-ASLI_6.3X7.7_DXL_; symbol Device:C_Small -> Device:C_Polarized
- C17: symbol Device:C_Small -> Device:C_Polarized
- D3: value 1N5819 -> SS14; footprint Diode_THT:D_DO-41_SOD81_P10.16mm_Horizontal -> Diode_SMD:D_SMA
Connections:
- net +12V: now also C15.1; no longer C15.2
- net CAN+: now also J15.2
- net CAN-: now also J15.1
- net GND: now also C15.2, C17.2, R17.2, R18.2, R19.2, R20.2, R21.2, R22.2, R23.2, R24.2, R25.2, R26.2; no longer C15.1, C17.1
- net MUX1: now also R17.1
- net MUX10: now also R26.1
- net MUX2: now also R18.1
- net MUX3: now also R19.1
- net MUX4: now also R20.1
- net MUX5: now also IC1.10 (IO17), R21.1; no longer IC1.16 (IO46)
- net MUX6: now also R22.1
- net MUX7: now also R23.1
- net MUX8: now also R24.1
- net MUX9: now also R25.1
- net VCC: now also C17.1; no longer C17.2
- no-connect marks 35 -> 33
Other:
- moved on the sheet: IC10, IC11, IC12, IC13, IC14, IC15, J10, J11, J12, J6, J7, J8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

Commit message: changed capacitor footprint, prolly something else too
Parts:
- C10: footprint Capacitor_SMD:C_0603_1608Metric -> Capacitor_SMD:C_1206_3216Metric

Commit message: Redesigned BMS Temp Board for 64 thermistors
Parts:
- removed IC10, IC11, IC12, IC13, IC14, IC15: CD74HC4067PWR, CD74HC4067PWR:TSSOP24_4P5X7P9_TEX, symbol CD74HC4067PWR:CD74HC4067PWR
- removed J10, J11, J6, J7, J8, J9: B32B-PUDSS-1_LF__SN_, ESP32_S3_WROOM_1_N8R8:JST_PUD_B32B-PUDSS_2x16_P2.00mm_Vertical_PN, symbol B32B-PUDSS-1_LF__SN_:B32B-PUDSS-1_LF__SN_
- removed R21, R22, R23, R24, R25, R26: 10k, Resistor_SMD:R_0603_1608Metric, symbol Device:R
Connections:
- net MUX10 is gone; now on net MUX1: IC1.21 (IO13)
- net MUX7 is gone; now on net MUX2: IC1.18 (IO10)
- net MUX8 is gone; now on net MUX3: IC1.19 (IO11)
- net MUX9 is gone; now on net MUX4: IC1.20 (IO12)
- net MUX1: no longer IC1.12 (IO8)
- net MUX2: no longer IC1.13 (IO19)
- net MUX3: no longer IC1.14 (IO20)
- net MUX4: no longer IC1.15 (IO3)
- net MUX5: no longer names the net of IC1.10 (IO17)
- net MUX6: no longer names the net of IC1.17 (IO9)
- no-connect marks 33 -> 39
Other:
- moved on the sheet: J12, J15, LED3, R16

Commit message: Changed temp board to use ampseal connector
Parts:
- removed J12, J14, J15: B2B-PH-K-S, B2B_PH_K_S:JST_B2B-PH-K-S, symbol B2B-PH-K-S:B2B-PH-K-S
- added J6: 776279-1, 776279_1:TE_776279-1, symbol 776279-1:776279-1
- LED3: value LED -> RED
Connections:
- net +12V: now also J6.2
- net +5V: now also J6.1
- net CAN+: now also J6.5
- net CAN-: now also J6.4
- net CHIP_PU: now also Q1.3 (C)
- net GND: now also J6.8
- net SHUTOFF: now also J6.3
- net SHUTDOWN_IND: now reaches IC1.10 (IO17)
- net SHUTDOWN_IND: now also R16.1
- net IO7: now reaches IC1.7 (IO7)
- net IO7: now also J6.6
- net IO15: now reaches IC1.8 (IO15)
- net IO15: now also J6.7
- no-connect marks 39 -> 36
Other:
- note added: "IO 7 and 15 are user-defined, use for whateva"
- note removed: "LED should be red"
- note removed: "Shutoff Signal Connector + Indicator"
- moved on the sheet: C11, C13, D1, IC3, LED1, LED3, R12, R15, R16, R2, U2

Commit message: Added Orion input to temp board
Parts:
- added R21: 10k, Resistor_SMD:R_0603_1608Metric, symbol Device:R
- added R22: 3.3k, Resistor_SMD:R_0603_1608Metric, symbol Device:R
Connections:
- net +12V: now also R21.1
- net GND: now also R22.2
- net IO7 renamed ORION
- net ORION: now also R21.2, R22.1

Commit message: Added optoisolator to shutoff signal output, updated BOM
Parts:
- added Q3: LTV-817S-TA1, LTV_817S_TA1:LTV-817S_LTO, symbol LTV_817S_TA1:LTV-817S-TA1
- added R23: 220, Resistor_SMD:R_0603_1608Metric, symbol Device:R
Connections:
- net +12V: now also Q3.4
- net GND: now also Q3.2
- net SHUTOFF: now also R23.1; no longer J6.3
- new net: Q3.1, R23.2
- new net SHUTOFF_ISO: J6.3, Q3.3
Other:
- note added: "Buck converter 12V->5V"
- note added: "Main I/O Connector"
- note added: "Multiplexers/Thermistor inputs"
- note added: "Shutoff signal isolation"
