File: BMS_Temp_Board/BMS_Temp_Board_V1.kicad_sch (KiCad schematic)
At the start: 71 parts, among them IC1 ESP32-S3-WROOM-1-N8R8, IC2 CP2102N-A02-GQFN28, IC3 TLP175A_TPL,E, IC4 TPS2116DRLR, IC5 MIC37100-3.3WS, IC6 CD74HC4067PWR, IC7 CD74HC4067PWR, IC8 CD74HC4067PWR, IC9 CD74HC4067PWR, J1 ESP_USB, J2 B32B-PUDSS-1_LF__SN_, J3 B32B-PUDSS-1_LF__SN_, J4 B32B-PUDSS-1_LF__SN_, J5 B32B-PUDSS-1_LF__SN_, J6 776279-1, Q1 MMBT2222LT1G, Q2 MMBT2222LT1G, Q3 LTV-817S-TA1, U1 USBLC6-2SC6, U2 SN65HVD230, U3 LM2575HVS-5.0_NOPB

Commit message: Added resistor and capacitor to optoisolator
Parts:
- added C16: 0.1uF, Capacitor_SMD:C_0603_1608Metric, symbol Device:C
- added R24: 10k, Resistor_SMD:R_0603_1608Metric, symbol Device:R
Connections:
- net +12V: now also R24.2; no longer Q3.4
- net GND: now also C16.2
- net SHUTOFF_ISO: now also C16.1
- new net: Q3.4, R24.1
