File: IMD Indicator/IMD Indicator.kicad_sch (KiCad schematic)
At the start: 11 parts, among them J1 172448-0004, J2 172448-0004, Q1 2N7002,215

Commit message: IMD Indicator
Parts:
- renumbered J2 to J1, J1 to J2
Changed lines of the file:
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@@
 		(dnp no)
 		(fields_autoplaced yes)
-		(property "Reference" "J2"
+		(property "Reference" "J1"
 			(at 115.57 38.1 0)
 			(effects
@@
 			(project "IMD Indicator"
 				(path "/2d398882-e4dd-424e-9a5b-db438ffb0a84"
-					(reference "J2")
+					(reference "J1")
 					(unit 1)
 				)
@@
 		(dnp no)
 		(fields_autoplaced yes)
-		(property "Reference" "J1"
+		(property "Reference" "J2"
 			(at 165.1 35.56 0)
 			(effects
@@
 			(project ""
 				(path "/2d398882-e4dd-424e-9a5b-db438ffb0a84"
-					(reference "J1")
-					(unit 1)
-				)
+					(reference "J2")
+					(unit 1)
+				)
