File: TSSI/TSSI/TSSI.kicad_sch (KiCad schematic)
At the start: 23 parts, among them J1 Conn_01x03_Socket, J2 B2P-VHLFSN, J3 B2P-VHLFSN, J4 B2P-VHLFSN, J5 B2P-VHLFSN, J6 B4P-VH, Q1 AO3400, Q2 AO3400, U1 ATtiny1614-SS, U2 MCP1703T-5002E/CB

Commit message: Changed chematic for cleanliness and some standardization issues
Connections:
- net +12V: now also C1.1; no longer C1.2
- net +5V: now also C2.2; no longer C2.1
- net GNDREF renamed GND
- net GND: now also C1.2, C2.1; no longer C1.1, C2.2
- no-connect marks 0 -> 7
Other:
- moved on the sheet: C1, C2, C3

Commit message: Changed resistor divider and trimmed board dimensions
Parts:
- R3, R7: value 4.7K -> 6.8k
Changed lines of the file:
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@@
 			)
 		)
-		(property "Value" "4.7K"
+		(property "Value" "6.8k"
 			(at 154.94 60.9599 0)
 			(effects
@@
 			)
 		)
-		(property "Value" "4.7K"
+		(property "Value" "6.8k"
 			(at 154.94 91.4399 0)
 			(effects
