File: sdm27ev/sdm27ev-vcu/hardware/sdm27ev-vcu-v1/vcu-power.kicad_sch (KiCad schematic)
At the start: 39 parts, among them IC1 TPD4E05U06QDQARQ1, IC2 TPS2121RUXR, IC3 TPS56637RPAR, IC4 TPS61023DRLT, J5 USB4725-03-C-KIT, Q1 RRL035P03FRATR, U3 HUSB238

Commit message: added all hierarchical sheet pins, added can termination optocouplers
Connections:
- net 5V renamed 5VA
