File: sdm27ev/sdm27ev-esf-tracive-system-schematics/Charging Shutdown Circuit.kicad_sch (KiCad schematic)
At the start: 10 parts, among them K11 1, K12 2, K5 AIR +, K6 AIR -, K7 Precharge, K9 Discharge

Commit message: updated esf tractive schematic to have msd
Changed lines of the file:
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@@
+	(polyline
+		(pts
+			(xy 114.3 40.64) (xy 114.3 48.26)
+		)
+		(stroke
+			(width 0)
+			(type default)
+		)
+	)
 	(polyline
 		(pts
@@
 		)
 	)
+	(polyline
+		(pts
+			(xy 106.68 40.64) (xy 114.3 40.64)
+		)
+		(stroke
+			(width 0)
+			(type default)
+		)
+	)
