File: sdm27ev/sdm27ev-esf-tracive-system-schematics/TS System Schematic.kicad_sch (KiCad schematic)
At the start: 2 parts

Commit message: updated esf tractive schematic to have msd
Other:
- note added: "MSD"
- note added: "Shutdown In"
- note added: "Shutdown Out"
- note removed: "NEED TO FIX"
